File: hardware/temp_sense_board/temp_sense_board.kicad_pcb (KiCad board)
At the start: 2 copper layers, 21.3 x 51.8 mm, 3 parts

Commit message: Updated PCB and Schematic
Parts:
- added I2C_EXTRA1: Conn_01x04_Socket, Connector_PinSocket_2.54mm:PinSocket_1x04_P2.54mm_Vertical, B.Cu at (100.5, 95.0)
- added I2C_EXTRA2: Conn_01x04_Socket, Connector_PinSocket_2.54mm:PinSocket_1x04_P2.54mm_Vertical, B.Cu at (94.5, 95.0)
- added I2C_EXTRA3: Conn_01x04_Socket, Connector_PinSocket_2.54mm:PinSocket_1x04_P2.54mm_Vertical, B.Cu at (94.5, 82.5)
- added I2C_EXTRA4: Conn_01x04_Socket, Connector_PinSocket_2.54mm:PinSocket_1x04_P2.54mm_Vertical, B.Cu at (100.5, 82.5)
Connections:
- net /GND renamed GND
- net /VBUS renamed VBUS
Routing:
- net SDA: track 31.9 -> 74.1 mm
- net SCL: track 33.5 -> 74.6 mm
Other:
- board size 21.3 x 51.8 mm -> 22.2 x 52.8 mm
